File: pcb/telegraph/telegraph.sch (KiCad schematic (older format))
At the start: 55 parts

Commit message: Finished annotated schematic; TODO source and footprint
Parts:
- C101: renamed from C?; value C_Small -> 10uF
- C102, C105, C106, C107, C115: renamed from C?; value C_Small -> 100nF
- R101, R104, R107: renamed from R?; value R_Small -> 10k
- R102, R103, R110: renamed from R?; value R_Small -> 470
- R108, R109, R111, R112, R116: renamed from R?; value R_Small -> 100k
- R114: renamed from R?; value 26.1k -> 26.1k 1%
- R117: renamed from R?; value 10k -> 10k 1%
- gave numbers to parts that had none: 35
Connections:
- no-connect marks 17 -> 26

Commit message: Save before autofill
Parts:
- added MH1, MH2, MH3, MH4: MountingHole, symbol Mechanical:MountingHole
- U1: renamed from U101; footprint (none) -> telegraph:TI_MSP430_QFN20
- renumbered C101 to C1, C110 to C10, C111 to C11, C112 to C12, C113 to C13, C114 to C14, C115 to C15, C102 to C2, C103 to C3, C104 to C4, C105 to C5, C106 to C6, C107 to C7, C108 to C8, C109 to C9, D101 to D1, D102 to D2, D103 to D3, J101 to J1, J102 to J2, J103 to J3, L101 to L1, Q101 to Q1, R101 to R1, R110 to R10, R111 to R11, R112 to R12, R113 to R13, R114 to R14, R115 to R15, R116 to R16, R117 to R17, R102 to R2, R103 to R3, R104 to R4, R105 to R5, R106 to R6, R107 to R7, R108 to R8, R109 to R9, TP101 to TP1, TP110 to TP10, TP102 to TP2, TP103 to TP3, TP104 to TP4, TP105 to TP5, TP106 to TP6, TP107 to TP7, TP108 to TP8, TP109 to TP9, U102 to U2, U103 to U3, Y101 to Y1
Connections:
- wire segments 139 -> 143

Commit message: Save before autofill; most parts sourced and autofill fixed
Parts:
- C1, C8: footprint (none) -> Capacitors_SMD:C_1206_HandSoldering; Mouser (none) -> 74-TMCMA1C106MTRF
- C10: value 0.1uF -> 100nF
- C11: footprint (none) -> Capacitors_SMD:C_0603_HandSoldering; Mouser (none) -> 77-VJ0603Y103KXAAC
- C13: footprint (none) -> Capacitors_SMD:C_1210_HandSoldering; Mouser (none) -> 581-TAJB226K016TNJ
- C15: footprint (none) -> Capacitors_SMD:C_1206_HandSoldering; Mouser (none) -> 77-VJ1206Y104KXXPBC
- C3: footprint (none) -> Capacitors_SMD:C_0402; Mouser (none) -> 81-GRM0225C1C100JA3L
- R10: footprint (none) -> Resistors_SMD:R_0603_HandSoldering; Mouser (none) -> 755-ESR03EZPJ471
- R11: footprint (none) -> Resistors_SMD:R_0402; Mouser (none) -> 755-SFR01MZPF1003
- R14: footprint (none) -> Resistors_SMD:R_0402; Mouser (none) -> 652-CR0402-FX2612GLF
- R17, R7: footprint (none) -> Resistors_SMD:R_0402; Mouser (none) -> 754-RR0510P-103D
- U1: Mouser (none) -> 595-430FR2512IRHLR
- Y1: value Crystal -> 32.768kHz; footprint (none) -> Crystals:Crystal_DS26_d2.0mm_l6.0mm_Horizontal
Connections:
- wire segments 143 -> 144
Changed lines of the file:
@@
 F 2 "telegraph:TI_MSP430_QFN20" H 2950 2900 50  0001 C CNN
 F 3 "" H 2950 2900 50  0001 C CNN
+F 4 "595-430FR2512IRHLR" H 2950 2900 50  0001 C CNN "Mouser"
 	2    2950 2900
 	-1   0    0    -1
@@
 P 5800 5750
 F 0 "C10" V 5571 5750 50  0000 C CNN
-F 1 "0.1uF" V 5662 5750 50  0000 C CNN
+F 1 "100nF" V 5662 5750 50  0000 C CNN
 F 2 "" H 5800 5750 50  0001 C CNN
 F 3 "~" H 5800 5750 50  0001 C CNN
@@
 F 0 "C11" H 4359 5804 50  0000 R CNN
 F 1 "10nF" H 4359 5895 50  0000 R CNN
-F 2 "" H 4450 5850 50  0001 C CNN
+F 2 "Capacitors_SMD:C_0603_HandSoldering" H 4450 5850 50  0001 C CNN
 F 3 "~" H 4450 5850 50  0001 C CNN
+F 4 "77-VJ0603Y103KXAAC" H 4450 5850 50  0001 C CNN "Mouser"
 	1    4450 5850
 	1    0    0    1
@@
 F 0 "C8" H 3158 5454 50  0000 R CNN
 F 1 "10uF 16V" H 3158 5545 50  0000 R CNN
-F 2 "" H 3250 5500 50  0001 C CNN
+F 2 "Capacitors_SMD:C_1206_HandSoldering" H 3250 5500 50  0001 C CNN
 F 3 "~" H 3250 5500 50  0001 C CNN
+F 4 "74-TMCMA1C106MTRF" H 3250 5500 50  0001 C CNN "Mouser"
 	1    3250 5500
 	-1   0    0    1
@@
 F 0 "R14" H 4909 6496 50  0000 L CNN
 F 1 "26.1k 1%" H 4909 6405 50  0000 L CNN
-F 2 "" H 4850 6450 50  0001 C CNN
+F 2 "Resistors_SMD:R_0402" H 4850 6450 50  0001 C CNN
 F 3 "~" H 4850 6450 50  0001 C CNN
+F 4 "652-CR0402-FX2612GLF" H 4850 6450 50  0001 C CNN "Mouser"
 	1    4850 6450
 	1    0    0    -1
@@
 F 0 "R17" H 4909 6796 50  0000 L CNN
 F 1 "10k 1%" H 4909 6705 50  0000 L CNN
-F 2 "" H 4850 6750 50  0001 C CNN
+F 2 "Resistors_SMD:R_0402" H 4850 6750 50  0001 C CNN
 F 3 "~" H 4850 6750 50  0001 C CNN
+F 4 "754-RR0510P-103D" H 4850 6750 50  0001 C CNN "Mouser"
 	1    4850 6750
 	1    0    0    -1
@@
 F 0 "C13" H 3792 6496 50  0000 L CNN
 F 1 "22uF" H 3792 6405 50  0000 L CNN
-F 2 "" H 3700 6450 50  0001 C CNN
+F 2 "Capacitors_SMD:C_1210_HandSoldering" H 3700 6450 50  0001 C CNN
 F 3 "~" H 3700 6450 50  0001 C CNN
+F 4 "581-TAJB226K016TNJ" H 3700 6450 50  0001 C CNN "Mouser"
 	1    3700 6450
 	1    0    0    -1
@@
 F 0 "R10" H 8959 4396 50  0000 L CNN
 F 1 "470" H 8959 4305 50  0000 L CNN
-F 2 "" H 8900 4350 50  0001 C CNN
+F 2 "Resistors_SMD:R_0603_HandSoldering" H 8900 4350 50  0001 C CNN
 F 3 "~" H 8900 4350 50  0001 C CNN
+F 4 "755-ESR03EZPJ471" H 8900 4350 50  0001 C CNN "Mouser"
 	1    8900 4350
 	0    -1   -1   0
@@
 F 0 "R11" H 7309 4546 50  0000 L CNN
 F 1 "100k" H 7309 4455 50  0000 L CNN
-F 2 "" H 7250 4500 50  0001 C CNN
+F 2 "Resistors_SMD:R_0402" H 7250 4500 50  0001 C CNN
 F 3 "~" H 7250 4500 50  0001 C CNN
+F 4 "755-SFR01MZPF1003" H 7250 4500 50  0001 C CNN "Mouser"
 	1    7250 4500
 	1    0    0    -1
@@
 F 0 "C1" V 4521 1200 50  0000 C CNN
 F 1 "10uF" V 4612 1200 50  0000 C CNN
-F 2 "" H 4750 1200 50  0001 C CNN
+F 2 "Capacitors_SMD:C_1206_HandSoldering" H 4750 1200 50  0001 C CNN
 F 3 "~" H 4750 1200 50  0001 C CNN
+F 4 "74-TMCMA1C106MTRF" V 4750 1200 50  0001 C CNN "Mouser"
 	1    4750 1200
 	0    1    1    0
@@
 F 0 "R7" H 6709 4196 50  0000 L CNN
 F 1 "10k" H 6709 4105 50  0000 L CNN
-F 2 "" H 6650 4150 50  0001 C CNN
+F 2 "Resistors_SMD:R_0402" H 6650 4150 50  0001 C CNN
 F 3 "~" H 6650 4150 50  0001 C CNN
+F 4 "754-RR0510P-103D" H 6650 4150 50  0001 C CNN "Mouser"
 	1    6650 4150
 	1    0    0    -1
@@
 P 4650 2150
 F 0 "Y1" H 4650 2418 50  0000 C CNN
-F 1 "Crystal" H 4650 2327 50  0000 C CNN
-F 2 "" H 4650 2150 50  0001 C CNN
+F 1 "32.768kHz" H 4650 2327 50  0000 C CNN
+F 2 "Crystals:Crystal_DS26_d2.0mm_l6.0mm_Horizontal" H 4650 2150 50  0001 C CNN
 F 3 "~" H 4650 2150 50  0001 C CNN
 F 4 "520-ECS327-6-13-X" H 4650 2150 50  0001 C CNN "Mouser"
@@
 F 0 "C3" H 4492 2396 50  0000 L CNN
 F 1 "10pF" H 4492 2305 50  0000 L CNN
-F 2 "" H 4400 2350 50  0001 C CNN
+F 2 "Capacitors_SMD:C_0402" H 4400 2350 50  0001 C CNN
 F 3 "~" H 4400 2350 50  0001 C CNN
+F 4 "81-GRM0225C1C100JA3L" H 4400 2350 50  0001 C CNN "Mouser"
 	1    4400 2350
 	1    0    0    -1
@@
 F 0 "C15" H 1692 6946 50  0000 L CNN
 F 1 "100nF" H 1692 6855 50  0000 L CNN
-F 2 "" H 1600 6900 50  0001 C CNN
+F 2 "Capacitors_SMD:C_1206_HandSoldering" H 1600 6900 50  0001 C CNN
 F 3 "~" H 1600 6900 50  0001 C CNN
+F 4 "77-VJ1206Y104KXXPBC" H 1600 6900 50  0001 C CNN "Mouser"
 	1    1600 6900
 	1    0    0    -1
@@
 	1    0    0    -1
 $EndComp
+$Comp
+L power:GND #PWR?
+U 1 1 5B69CB06
+P 4600 6150
+F 0 "#PWR?" H 4600 5900 50  0001 C CNN
+F 1 "GND" V 4605 6022 50  0000 R CNN
+F 2 "" H 4600 6150 50  0001 C CNN
+F 3 "" H 4600 6150 50  0001 C CNN
+	1    4600 6150
+	0    1    1    0
+$EndComp
+Wire Wire Line
+	4600 6150 4700 6150
 $EndSCHEMATC

Commit message: Most parts sourced
Parts:
- C10, C2, C5, C6, C7: footprint (none) -> Capacitors_SMD:C_1206_HandSoldering; Mouser (none) -> 77-VJ1206Y104KXXPBC
- C12: footprint (none) -> Capacitors_SMD:C_0402; Mouser (none) -> 710-885012205047
- C14: footprint (none) -> Capacitors_SMD:C_1210_HandSoldering; Mouser (none) -> 581-TAJB226K016TNJ
- C4: footprint (none) -> Capacitors_SMD:C_0402; Mouser (none) -> 81-GRM0225C1C100JA3L
- C9: footprint (none) -> Capacitors_SMD:C_1206_HandSoldering; Mouser (none) -> 74-TMCMA1C106MTRF
- D1, D2, D3: footprint (none) -> LEDs:LED_0603_HandSoldering; Mouser (none) -> 710-150060VS75000
- J1: footprint (none) -> Socket_Strips:Socket_Strip_Straight_2x02_Pitch2.54mm
- J2, J3: footprint (none) -> Socket_Strips:Socket_Strip_Straight_1x02_Pitch2.54mm; Mouser (none) -> NoPart
- L1: footprint (none) -> Inductors:Inductor_Taiyo-Yuden_NR-24xx_HandSoldering; Mouser (none) -> 963-NRH2410T4R7MN
- MH1, MH2, MH3, MH4: footprint (none) -> Mounting_Holes:MountingHole_4.3mm_M4_Pad; Mouser (none) -> NoPart
- R1, R4: footprint (none) -> Resistors_SMD:R_0402; Mouser (none) -> 754-RR0510P-103D
- R12, R13, R16, R8, R9: footprint (none) -> Resistors_SMD:R_0402; Mouser (none) -> 755-SFR01MZPF1003
- R15: footprint (none) -> Resistors_SMD:R_0603_HandSoldering; Mouser (none) -> 71-CRCW060313K0FKEAC
- R2, R3, R5, R6: footprint (none) -> Resistors_SMD:R_0603_HandSoldering; Mouser (none) -> 755-ESR03EZPJ471
- TP1, TP10, TP2, TP3, TP4, TP5, TP6, TP7, TP8, TP9: footprint (none) -> Measurement_Points:Measurement_Point_Round-SMD-Pad_Small; Mouser (none) -> NoPart
- U3: footprint (none) -> telegraph:Diodes_SO8EP

Commit message: All components sourced
Parts:
- removed Q1: Q_PMOS_DGS, symbol Device:Q_PMOS_DGS
- added Q1: RU1E002SPTCL, telegraph:Rohm_UMT3F, symbol Device:Q_PMOS_GSD
- J1: Mouser (none) -> NoPart
Changed lines of the file:
@@
 F 2 "Socket_Strips:Socket_Strip_Straight_2x02_Pitch2.54mm" H 8600 5300 50  0001 C CNN
 F 3 "~" H 8600 5300 50  0001 C CNN
+F 4 "NoPart" H 8600 5300 50  0001 C CNN "Mouser"
 	1    8600 5300
 	1    0    0    -1
@@
 Wire Wire Line
 	2550 5450 2450 5450
-$Comp
-L Device:Q_PMOS_DGS Q1
-U 1 1 5B6C13A0
-P 2900 5450
-F 0 "Q1" V 3243 5450 50  0000 C CNN
-F 1 "Q_PMOS_DGS" V 3152 5450 50  0000 C CNN
-F 2 "" H 3100 5550 50  0001 C CNN
-F 3 "~" H 2900 5450 50  0001 C CNN
-	1    2900 5450
-	0    -1   -1   0
-$EndComp
 Wire Wire Line
 	3100 5350 3250 5350
@@
 $EndComp
 $Comp
-L power:GND #PWR?
+L power:GND #PWR0101
 U 1 1 5B69CB06
 P 4600 6150
-F 0 "#PWR?" H 4600 5900 50  0001 C CNN
+F 0 "#PWR0101" H 4600 5900 50  0001 C CNN
 F 1 "GND" V 4605 6022 50  0000 R CNN
 F 2 "" H 4600 6150 50  0001 C CNN
@@
 Wire Wire Line
 	4600 6150 4700 6150
+$Comp
+L Device:Q_PMOS_GSD Q1
+U 1 1 5B6BBBD4
+P 2900 5450
+F 0 "Q1" V 3243 5450 50  0000 C CNN
+F 1 "RU1E002SPTCL" V 3152 5450 50  0000 C CNN
+F 2 "telegraph:Rohm_UMT3F" H 3100 5550 50  0001 C CNN
+F 3 "~" H 2900 5450 50  0001 C CNN
+F 4 "755-RU1E002SPTCL" V 2900 5450 50  0001 C CNN "Mouser"
+	1    2900 5450
+	0    -1   -1   0
+$EndComp
 $EndSCHEMATC

Commit message: Layout finished; need to move silkscreens around now
Parts:
- removed J3: Conn_01x02, Socket_Strips:Socket_Strip_Straight_1x02_Pitch2.54mm, symbol Connector_Generic:Conn_01x02
- removed MH3, MH4: MountingHole, Mounting_Holes:MountingHole_4.3mm_M4_Pad, symbol Mechanical:MountingHole
- added SW1: SW_SPST, Socket_Strips:Socket_Strip_Straight_1x02_Pitch2.54mm, symbol Switch:SW_SPST
- U2: footprint RF_Module:RN42 -> RF_Modules:RN42
Connections:
- wire segments 144 -> 146
Changed lines of the file:
@@
 F 0 "U2" H 8300 3667 50  0000 C CNN
 F 1 "RN42" H 8300 3576 50  0000 C CNN
-F 2 "RF_Module:RN42" H 8250 3450 50  0001 C CNN
+F 2 "RF_Modules:RN42" H 8250 3450 50  0001 C CNN
 F 3 "http://ww1.microchip.com/downloads/en/DeviceDoc/rn-42-ds-v2.32r.pdf" H 8300 1800 50  0001 C CNN
 F 4 "765-RN42HID-I/RM" H 8300 2600 50  0001 C CNN "Mouser"
@@
 RN42_CTS
 $Comp
-L Connector_Generic:Conn_01x02 J3
-U 1 1 5B6FEE88
-P 2300 6850
-F 0 "J3" H 2380 6842 50  0000 L CNN
-F 1 "Conn_01x02" H 2380 6751 50  0000 L CNN
-F 2 "Socket_Strips:Socket_Strip_Straight_1x02_Pitch2.54mm" H 2300 6850 50  0001 C CNN
-F 3 "~" H 2300 6850 50  0001 C CNN
-F 4 "NoPart" H 2300 6850 50  0001 C CNN "Mouser"
-	1    2300 6850
-	1    0    0    -1
-$EndComp
-$Comp
 L Device:R_Small R16
 U 1 1 5B6FF396
@@
 	2050 6750 1600 6750
 Wire Wire Line
-	2050 6850 2050 6750
-Wire Wire Line
-	2100 6850 2050 6850
-Wire Wire Line
-	2050 6950 2100 6950
-Wire Wire Line
-	2050 7050 2050 6950
-Wire Wire Line
 	1600 7050 2050 7050
 Connection ~ 1600 7050
@@
 	1750 5450 1750 5550
 $Comp
-L Mechanical:MountingHole MH4
-U 1 1 5B6A1719
-P 1500 4850
-F 0 "MH4" H 1600 4896 50  0000 L CNN
-F 1 "MountingHole" H 1600 4805 50  0000 L CNN
-F 2 "Mounting_Holes:MountingHole_4.3mm_M4_Pad" H 1500 4850 50  0001 C CNN
-F 3 "~" H 1500 4850 50  0001 C CNN
-F 4 "NoPart" H 1500 4850 50  0001 C CNN "Mouser"
-	1    1500 4850
-	1    0    0    -1
-$EndComp
-$Comp
 L Mechanical:MountingHole MH2
 U 1 1 5B6A1847
@@
 F 4 "NoPart" H 1500 4600 50  0001 C CNN "Mouser"
 	1    1500 4600
-	1    0    0    -1
-$EndComp
-$Comp
-L Mechanical:MountingHole MH3
-U 1 1 5B6A1922
-P 850 4850
-F 0 "MH3" H 950 4896 50  0000 L CNN
-F 1 "MountingHole" H 950 4805 50  0000 L CNN
-F 2 "Mounting_Holes:MountingHole_4.3mm_M4_Pad" H 850 4850 50  0001 C CNN
-F 3 "~" H 850 4850 50  0001 C CNN
-F 4 "NoPart" H 850 4850 50  0001 C CNN "Mouser"
-	1    850  4850
 	1    0    0    -1
 $EndComp
@@
 	0    -1   -1   0
 $EndComp
+Wire Wire Line
+	2050 6750 2050 6600
+Wire Wire Line
+	2050 6600 2300 6600
+Wire Wire Line
+	2300 6600 2300 6700
+Wire Wire Line
+	2050 7050 2050 7200
+Wire Wire Line
+	2050 7200 2300 7200
+Wire Wire Line
+	2300 7200 2300 7100
+$Comp
+L Switch:SW_SPST SW1
+U 1 1 5B6CF995
+P 2300 6900
+F 0 "SW1" V 2254 6998 50  0000 L CNN
+F 1 "SW_SPST" V 2345 6998 50  0000 L CNN
+F 2 "Socket_Strips:Socket_Strip_Straight_1x02_Pitch2.54mm" H 2300 6900 50  0001 C CNN
+F 3 "" H 2300 6900 50  0001 C CNN
+F 4 "NoPart" V 2300 6900 50  0001 C CNN "Mouser"
+	1    2300 6900
+	0    1    1    0
+$EndComp
 $EndSCHEMATC

Commit message: Finish PCB board
Parts:
- added C16: 1nF, Capacitors_SMD:C_0603_HandSoldering, symbol Device:C_Small
- added C17: 1uF, Capacitors_SMD:C_0805_HandSoldering, symbol Device:C_Small
- added R18, R19: 100k, Resistors_SMD:R_0402, symbol Device:R_Small
Connections:
- wire segments 146 -> 158
- no-connect marks 26 -> 25
Changed lines of the file:
@@
 NoConn ~ 4050 3200
 NoConn ~ 4050 3300
-NoConn ~ 4050 3800
 NoConn ~ 4050 3900
 NoConn ~ 4050 4000
@@
 	0    1    1    0
 $EndComp
+Text Label 6400 1350 2    50   ~ 0
+SWBTDIO
+$Comp
+L Device:R_Small R18
+U 1 1 5B6DBF18
+P 6400 1150
+F 0 "R18" H 6459 1196 50  0000 L CNN
+F 1 "100k" H 6459 1105 50  0000 L CNN
+F 2 "Resistors_SMD:R_0402" H 6400 1150 50  0001 C CNN
+F 3 "~" H 6400 1150 50  0001 C CNN
+F 4 "755-SFR01MZPF1003" H 6400 1150 50  0001 C CNN "Mouser"
+	1    6400 1150
+	1    0    0    -1
+$EndComp
+$Comp
+L Device:R_Small R19
+U 1 1 5B6DC26E
+P 6750 1150
+F 0 "R19" H 6809 1196 50  0000 L CNN
+F 1 "100k" H 6809 1105 50  0000 L CNN
+F 2 "Resistors_SMD:R_0402" H 6750 1150 50  0001 C CNN
+F 3 "~" H 6750 1150 50  0001 C CNN
+F 4 "755-SFR01MZPF1003" H 6750 1150 50  0001 C CNN "Mouser"
+	1    6750 1150
+	1    0    0    -1
+$EndComp
+Wire Wire Line
+	6400 1250 6400 1300
+Wire Wire Line
+	6750 1250 6750 1300
+Wire Wire Line
+	6750 1300 6400 1300
+Connection ~ 6400 1300
+Wire Wire Line
+	6400 1300 6400 1350
+Wire Wire Line
+	6400 950  6400 1000
+Wire Wire Line
+	6400 1000 6750 1000
+Wire Wire Line
+	6750 1000 6750 1050
+Connection ~ 6400 1000
+Wire Wire Line
+	6400 1000 6400 1050
+Text Label 6400 950  0    50   ~ 0
++3V3
+$Comp
+L Device:C_Small C16
+U 1 1 5B6F6CB4
+P 6400 1450
+F 0 "C16" H 6492 1496 50  0000 L CNN
+F 1 "1nF" H 6492 1405 50  0000 L CNN
+F 2 "Capacitors_SMD:C_0603_HandSoldering" H 6400 1450 50  0001 C CNN
+F 3 "~" H 6400 1450 50  0001 C CNN
+F 4 "77-VJ0603Y102JXJPBC" H 6400 1450 50  0001 C CNN "Mouser"
+	1    6400 1450
+	1    0    0    -1
+$EndComp
+$Comp
+L power:GND #PWR0102
+U 1 1 5B6F6F8B
+P 6400 1600
+F 0 "#PWR0102" H 6400 1350 50  0001 C CNN
+F 1 "GND" H 6405 1427 50  0000 C CNN
+F 2 "" H 6400 1600 50  0001 C CNN
+F 3 "" H 6400 1600 50  0001 C CNN
+	1    6400 1600
+	1    0    0    -1
+$EndComp
+Wire Wire Line
+	6400 1550 6400 1600
+$Comp
+L Device:C_Small C17
+U 1 1 5B6FF4B6
+P 4500 4000
+F 0 "C17" H 4592 4046 50  0000 L CNN
+F 1 "1uF" H 4592 3955 50  0000 L CNN
+F 2 "Capacitors_SMD:C_0805_HandSoldering" H 4500 4000 50  0001 C CNN
+F 3 "~" H 4500 4000 50  0001 C CNN
+F 4 "603-CC805MKX7R6BB105" H 4500 4000 50  0001 C CNN "Mouser"
+	1    4500 4000
+	1    0    0    -1
+$EndComp
+Wire Wire Line
+	4050 3800 4500 3800
+Wire Wire Line
+	4500 3800 4500 3900
+$Comp
+L power:GND #PWR031
+U 1 1 5B7067AA
+P 4500 4200
+F 0 "#PWR031" H 4500 3950 50  0001 C CNN
+F 1 "GND" H 4505 4027 50  0000 C CNN
+F 2 "" H 4500 4200 50  0001 C CNN
+F 3 "" H 4500 4200 50  0001 C CNN
+	1    4500 4200
+	1    0    0    -1
+$EndComp
+Wire Wire Line
+	4500 4100 4500 4200
 $EndSCHEMATC

Commit message: Replace RN42 RC pair with one easier to drive from MCU
Parts:
- C7: value 100nF -> 10nF; footprint Capacitors_SMD:C_1206_HandSoldering -> Capacitors_SMD:C_0603_HandSoldering; Mouser 77-VJ1206Y104KXXPBC -> 77-VJ0603Y103KXAAC
- R7: value 10k -> 100k; Mouser 754-RR0510P-103D -> 755-SFR01MZPF1003
Changed lines of the file:
@@
 Text Label 5150 3400 2    50   ~ 0
 RN42_RSTN
-$Comp
-L Device:R_Small R7
-U 1 1 5B7646C1
-P 6650 4150
-F 0 "R7" H 6709 4196 50  0000 L CNN
-F 1 "10k" H 6709 4105 50  0000 L CNN
-F 2 "Resistors_SMD:R_0402" H 6650 4150 50  0001 C CNN
-F 3 "~" H 6650 4150 50  0001 C CNN
-F 4 "754-RR0510P-103D" H 6650 4150 50  0001 C CNN "Mouser"
-	1    6650 4150
-	1    0    0    -1
-$EndComp
-$Comp
-L Device:C_Small C7
-U 1 1 5B7648D9
-P 6650 4500
-F 0 "C7" H 6742 4546 50  0000 L CNN
-F 1 "100nF" H 6742 4455 50  0000 L CNN
-F 2 "Capacitors_SMD:C_1206_HandSoldering" H 6650 4500 50  0001 C CNN
-F 3 "~" H 6650 4500 50  0001 C CNN
-F 4 "77-VJ1206Y104KXXPBC" H 6650 4500 50  0001 C CNN "Mouser"
-	1    6650 4500
-	1    0    0    -1
-$EndComp
 Wire Wire Line
 	6650 4250 6650 4400
@@
 Wire Wire Line
 	4500 4100 4500 4200
+$Comp
+L Device:R_Small R7
+U 1 1 5B6B6137
+P 6650 4150
+F 0 "R7" H 6709 4196 50  0000 L CNN
+F 1 "100k" H 6709 4105 50  0000 L CNN
+F 2 "Resistors_SMD:R_0402" H 6650 4150 50  0001 C CNN
+F 3 "~" H 6650 4150 50  0001 C CNN
+F 4 "755-SFR01MZPF1003" H 6650 4150 50  0001 C CNN "Mouser"
+	1    6650 4150
+	1    0    0    -1
+$EndComp
+$Comp
+L Device:C_Small C7
+U 1 1 5B6B62CA
+P 6650 4500
+F 0 "C7" H 6559 4454 50  0000 R CNN
+F 1 "10nF" H 6559 4545 50  0000 R CNN
+F 2 "Capacitors_SMD:C_0603_HandSoldering" H 6650 4500 50  0001 C CNN
+F 3 "~" H 6650 4500 50  0001 C CNN
+F 4 "77-VJ0603Y103KXAAC" H 6650 4500 50  0001 C CNN "Mouser"
+	1    6650 4500
+	-1   0    0    1
+$EndComp
 $EndSCHEMATC
